Commit message: my robot properties fix

File: src/my_robot_description/urdf/macros.xacro (robot description, xacro)
@@ -56,5 +56,5 @@
         		rpy="${-tY*PI/2} 0 0" />
         <mass value="${wheelMass}"/>
-        <cylinder_inertia
+        <xacro:cylinder_inertia
           m="${wheelMass}"
           r="${wheelRadius}"

File: src/my_robot_description/urdf/my_robot.xacro (robot description, xacro)
@@ -42,5 +42,5 @@
 					rpy="0 0 0"/>
 			<mass value="${chassisMass}"/>
-			<box_inertia
+			<xacro:box_inertia
 				m="${chassisMass}"
 				x="${chassisLength}"
@@ -73,11 +73,11 @@
 					rpy="0 0 0"/>
 			<mass value="${casterMass}"/>
-			<sphere_inertia
+			<xacro:sphere_inertia
 				m="${casterMass}"
 				r="${casterRadius}"/>
 		</inertial>
 	</link>
-	<wheel lr="left" tY="-1"/>
-	<wheel lr="right" tY="1"/>
+	<xacro:wheel lr="left" tY="-1"/>
+	<xacro:wheel lr="right" tY="1"/>
 	<!-- Sensor models -->
 	<xacro:include filename="$(find my_robot_description)/urdf/sensors.xacro" />

File: src/my_robot_description/urdf/my_robot_properties.xacro (robot description, xacro)
@@ -5,6 +5,6 @@
 	<!-- Chassis properties -->
 	<xacro:property name="chassisHeight" value="0.0623"/>
-	<xacro:property name="chassisLength" value="0.255"/>
-	<xacro:property name="chassisWidth" value="0.162"/>
+	<xacro:property name="chassisLength" value="0.198"/>
+	<xacro:property name="chassisWidth" value="0.119"/>
 	<xacro:property name="chassisMass" value="0.15"/>
 	<!-- Caster wheel properties -->
@@ -13,13 +13,13 @@
 	<xacro:property name="casterOffsetX" value="0.091"/>
 	<!-- Differential-drive wheels properties -->
-	<xacro:property name="wheelWidth" value="0.04"/>
-	<xacro:property name="wheelRadius" value="0.022"/>
+	<xacro:property name="wheelWidth" value="0.026"/>
+	<xacro:property name="wheelRadius" value="0.032"/>
 	<xacro:property name="wheelMass" value="0.05"/>
-	<xacro:property name="wheelOffsetY" value="0.0"/>
+	<xacro:property name="wheelOffsetY" value="0.037"/>
 	<!-- Hokuyo laser properties -->
 	<xacro:property name="hokuyoMass" value="0.01"/>
-	<xacro:property name="hokuyoLength" value="0.095"/>
-	<xacro:property name="hokuyoWidth" value="0.065"/>
-	<xacro:property name="hokuyoHeight" value="0.06"/>
+	<xacro:property name="hokuyoLength" value="0.05"/>
+	<xacro:property name="hokuyoWidth" value="0.05"/>
+	<xacro:property name="hokuyoHeight" value="0.07"/>
 	<xacro:property name="hokuyoOffsetX" value="0.035"/>
 	<!--xacro:property name="hokuyoOffsetX" value="0.05"/-->
@@ -27,7 +27,7 @@
 	<!--xacro:property name="hokuyoOffsetZ" value="0.1125"/-->
 	<!-- Camera properties -->
-	<xacro:property name="cameraLength" value="0.045"/>
-	<xacro:property name="cameraWidth" value="0.04"/>
-	<xacro:property name="cameraHeight" value="0.04"/>
+	<xacro:property name="cameraLength" value="0.04"/>
+	<xacro:property name="cameraWidth" value="0.08"/>
+	<xacro:property name="cameraHeight" value="0.03"/>
 	<xacro:property name="cameraMass" value="0.01"/>
 	<xacro:property name="cameraOffsetX" value="0.095"/>

File: src/my_robot_description/urdf/sensors.xacro (robot description, xacro)
@@ -39,5 +39,5 @@
       <origin xyz="0 0 0"
               rpy="0 0 0"/>
-      <box_inertia m="${cameraMass}"
+      <xacro:box_inertia m="${cameraMass}"
                    x="${cameraLength}"
                    y="${cameraWidth}"
@@ -81,5 +81,5 @@
       <origin xyz="0 0 0"
               rpy="0 0 0"/>
-      <box_inertia
+      <xacro:box_inertia
         m="${hokuyoMass}"
         x="${hokuyoLength}"
