Commit message: Update mike_robot.xacro

File: src/mastering_ros_robot_description_pkg/urdf/mike_robot.xacro (robot description, xacro)
@@ -96,19 +96,19 @@
   <!-- SENSORS -->
   <!-- hokuyo -->
-<!--  <link name="hokuyo_link">-->
-<!--    <visual>-->
-<!--      <origin xyz="0 0 0" rpy="0 0 0" />-->
-<!--      <geometry>-->
-<!--        <box size="${hokuyo_size} ${hokuyo_size} ${hokuyo_size}"/>-->
-<!--      </geometry>-->
-<!--      <material name="Blue" />-->
-<!--    </visual>-->
-<!--  </link>-->
-<!--  <joint name="hokuyo_joint" type="fixed">-->
-<!--    <origin xyz="${base_radius - hokuyo_size/2} 0 ${base_height+hokuyo_size/4}" rpy="0 0 0" />-->
-<!--    <parent link="base_link"/>-->
-<!--    <child link="hokuyo_link" />-->
-<!--  </joint>-->
-  <xacro:include filename="$(find ydlidar_ros)/urdf/ydlidar.urdf" />
+  <link name="hokuyo_link">
+    <visual>
+      <origin xyz="0 0 0" rpy="0 0 0" />
+      <geometry>
+        <box size="${hokuyo_size} ${hokuyo_size} ${hokuyo_size}"/>
+      </geometry>
+      <material name="Blue" />
+    </visual>
+  </link>
+  <joint name="hokuyo_joint" type="fixed">
+    <origin xyz="${base_radius - hokuyo_size/2} 0 ${base_height+hokuyo_size/4}" rpy="0 0 0" />
+    <parent link="base_link"/>
+    <child link="hokuyo_link" />
+  </joint>
+<!--  <xacro:include filename="$(find ydlidar_ros)/urdf/ydlidar.urdf" />-->
   <gazebo reference="base_laser">
     <material>Gazebo/Blue</material>
